File: ARDUINO-MICRO.sch (KiCad schematic (older format))
At the start: 48 parts, among them P4 ICSP, P5 USB-MICRO, P6 RS232, SW1 SW_PUSH, U2 ATmega32U4, U3 ADM3101EACPZ-250R7, Y1 16MHz

Commit message: Update
Parts:
- removed D2: BLUE, symbol device:LED
- removed D6: GREEN, symbol device:LED
- removed R11, R18: 1k, Resistor_SMD:R_0603_1608Metric, symbol device:R
- added C24: 100nF 6.3V, Capacitor_SMD:C_0603_1608Metric, symbol device:C
- added R21: R DNM, Resistor_SMD:R_0603_1608Metric, symbol device:R
- D8: renamed from D5; value YELLOW -> GREEN
- gave numbers to parts that had none: 1
- renumbered C24 to C25, C25 to C26, D1 to D5, D3 to D6, D4 to D7, R10 to R14, R12 to R15, R13 to R16, R14 to R17, R15 to R18, R16 to R19, R17 to R20, R24 to R22, R19 to R24, R20 to R27, R21 to R28, R22 to R29, R23 to R30
Connections:
- net labels added: +5V
- net labels removed: VDD
- wire segments 186 -> 198

Commit message: Update
Parts:
- C11, C12, C13, C14, C15, C16, C17, C18, C19, C20, C21, C22, C23, C24, C26: symbol device:C -> Driverino-rescue:C-device
- C25: symbol device2:CT -> Driverino-rescue:CT-device2
- D5: symbol device:DIODE -> Driverino-rescue:DIODE-device
- D6, D8: symbol device:LED -> Driverino-rescue:LED-device
- D7: symbol device:ZENERsmall -> Driverino-rescue:ZENERsmall-device
- F1: symbol device:FUSE -> Driverino-rescue:FUSE-device
- L2: symbol device:INDUCTOR_SMALL -> Driverino-rescue:INDUCTOR_SMALL-device
- P4: symbol conn:CONN_3X2 -> Driverino-rescue:CONN_3X2-conn
- P5: symbol conn:CONN_5 -> Driverino-rescue:CONN_5-conn
- P6: symbol conn:CONN_3 -> Driverino-rescue:CONN_3-conn
- R14, R15, R16, R17, R18, R19, R20, R21, R22, R23, R24, R25, R26, R27, R28, R29, R30: symbol device:R -> Driverino-rescue:R-device
- SW1: symbol device:SW_PUSH -> Driverino-rescue:SW_PUSH-device
- U2: symbol V2-30A110-A-symbols:ATmega32U4 -> Driverino-rescue:ATmega32U4-V2-30A110-A-symbols
- U3: symbol ad:ADM3101EACPZ-250R7 -> Driverino-rescue:ADM3101EACPZ-250R7-ad
- Y1: symbol device:CRYSTAL -> Driverino-rescue:CRYSTAL-device

Commit message: Update
Parts:
- removed C25: 22uF, symbol Driverino-rescue:CT-device2
- removed D8: GREEN, symbol Driverino-rescue:LED-device
- removed R19: 1k, Resistor_SMD:R_0603_1608Metric, symbol Driverino-rescue:R-device
- removed R22: 10k, Resistor_SMD:R_0402_1005Metric, symbol Driverino-rescue:R-device
- added C15: 10uF, Capacitor_SMD:C_1206_3216Metric, symbol Driverino-rescue:C-device
- added D3: GREEN, LED_SMD:LED_0603_1608Metric, symbol Driverino-rescue:LED-device
- added JP1: VCC_SEL, Driverino:TDD01H0SB1R, symbol Jumper:Jumper_3_Bridged12
- added P1: RC_IN, Connector_PinHeader_2.54mm:PinHeader_1x03_P2.54mm_Horizontal, symbol Driverino-rescue:CONN_3-conn
- added R11: 0R DNM, Resistor_SMD:R_0402_1005Metric, symbol Driverino-rescue:R-device
- added R3: 1k, Resistor_SMD:R_0402_1005Metric, symbol Driverino-rescue:R-device
- C1: renamed from C11; footprint Capacitor_SMD:C_0603_1608Metric -> Capacitor_SMD:C_0402_1005Metric; Manufacturer (none) -> Murata; P/N C0603C104K4RAC -> (none); Provider (none) -> Mouser; ProviderCode (none) -> 81-GCM155R71H104KE2J; manf# (none) -> GCM155R71H104KE02J
- C10: renamed from C20; P/N GRM1555C1H180JA01D -> (none); Productor Murata -> (none)
- C11: renamed from C21; P/N GRM1555C1H180JA01D -> (none); Productor Murata -> (none)
- C12: renamed from C22; value 0.1uF 16V 10% -> 100nF; footprint Capacitor_SMD:C_0603_1608Metric -> Capacitor_SMD:C_0402_1005Metric; Manufacturer (none) -> Murata; P/N C0603C104K4RAC -> (none); Provider (none) -> Mouser; ProviderCode (none) -> 81-GCM155R71H104KE2J; manf# (none) -> GCM155R71H104KE02J
- C13: renamed from C23; value 0.1uF 16V 10% -> 100nF; footprint Capacitor_SMD:C_0603_1608Metric -> Capacitor_SMD:C_0402_1005Metric; Manufacturer (none) -> Murata; P/N C0603C104K4RAC -> (none); Provider (none) -> Mouser; ProviderCode (none) -> 81-GCM155R71H104KE2J; manf# (none) -> GCM155R71H104KE02J
- C14: renamed from C24; value 100nF 6.3V -> 100nF; footprint Capacitor_SMD:C_0603_1608Metric -> Capacitor_SMD:C_0402_1005Metric; Manufacturer (none) -> Murata; Provider (none) -> Mouser; ProviderCode (none) -> 81-GCM155R71H104KE2J; manf# (none) -> GCM155R71H104KE02J
- C16: renamed from C26; footprint Capacitor_SMD:C_0603_1608Metric -> Capacitor_SMD:C_0402_1005Metric; Manufacturer (none) -> Murata; Provider (none) -> Mouser; ProviderCode (none) -> 81-GCM155R71H104KE2J; manf# (none) -> GCM155R71H104KE02J
- C2: renamed from C12; footprint Capacitor_SMD:C_0603_1608Metric -> Capacitor_SMD:C_0402_1005Metric; Manufacturer (none) -> Murata; P/N C0603C104K4RAC -> (none); Provider (none) -> Mouser; ProviderCode (none) -> 81-GCM155R71H104KE2J; manf# (none) -> GCM155R71H104KE02J
- C3: renamed from C13; value 1uF 16V 10% -> 1uF; Manufacturer (none) -> AVX; P/N C0603C105K4PACTU -> (none); Provider (none) -> Mouser; ProviderCode (none) -> 581-0603DC105MAT2A; manf# (none) -> 0603DC105MAT2A
- C4: renamed from C14; value 1uF 16V 10% -> 1uF; Manufacturer (none) -> AVX; P/N C0603C105K4PACTU -> (none); Provider (none) -> Mouser; ProviderCode (none) -> 581-0603DC105MAT2A; manf# (none) -> 0603DC105MAT2A
- C5: renamed from C15; value 0.1uF 16V 10% -> 100nF; footprint Capacitor_SMD:C_0603_1608Metric -> Capacitor_SMD:C_0402_1005Metric; Manufacturer (none) -> Murata; P/N C0603C104K4RAC -> (none); Provider (none) -> Mouser; ProviderCode (none) -> 81-GCM155R71H104KE2J; manf# (none) -> GCM155R71H104KE02J
- C6: renamed from C16; value 100nF 6.3V -> 100nF; footprint Capacitor_SMD:C_0603_1608Metric -> Capacitor_SMD:C_0402_1005Metric; Manufacturer (none) -> Murata; Provider (none) -> Mouser; ProviderCode (none) -> 81-GCM155R71H104KE2J; manf# (none) -> GCM155R71H104KE02J
- C7: renamed from C17; value 0.1uF 16V 10% -> 100nF; footprint Capacitor_SMD:C_0603_1608Metric -> Capacitor_SMD:C_0402_1005Metric; Manufacturer (none) -> Murata; P/N C0603C104K4RAC -> (none); Provider (none) -> Mouser; ProviderCode (none) -> 81-GCM155R71H104KE2J; manf# (none) -> GCM155R71H104KE02J
- C8: renamed from C18; value 100nF 16V 10% -> 100nF; footprint Capacitor_SMD:C_0603_1608Metric -> Capacitor_SMD:C_0402_1005Metric; Manufacturer (none) -> Murata; P/N C0603C104K4RAC -> (none); Provider (none) -> Mouser; ProviderCode (none) -> 81-GCM155R71H104KE2J; manf# (none) -> GCM155R71H104KE02J
- C9: renamed from C19; value 0.1uF 16V 10% -> 100nF; footprint Capacitor_SMD:C_0603_1608Metric -> Capacitor_SMD:C_0402_1005Metric; Manufacturer (none) -> Murata; P/N C0603C104K4RAC -> (none); Provider (none) -> Mouser; ProviderCode (none) -> 81-GCM155R71H104KE2J; manf# (none) -> GCM155R71H104KE02J
- D1: renamed from D5; footprint (none) -> Diode_SMD:D_0402_1005Metric; Manufacturer (none) -> Comchip; Provider (none) -> Mouser; ProviderCode (none) -> 750-CDBQR70; manf# (none) -> CDBQR70-HF
- D2: renamed from D6; footprint (none) -> LED_SMD:LED_0603_1608Metric; Manufacturer (none) -> Kingbright; Provider (none) -> Mouser; ProviderCode (none) -> 604-APT1608YC; manf# (none) -> APT1608YC
- D4: renamed from D7; value VZ=3V -> VZ=5V; footprint Diode_SMD:D_SOD-523 -> Diode_SMD:D_SOD-123; P/N BZX585-B3V3 -> (none); Productor Nexperia -> (none); Provider (none) -> Mouser; ProviderCode (none) -> 771-BZT52-C4V7X; manf# BZX585-B3V3 -> BZT52-C4V7X
- F1: footprint Resistor_SMD:R_1812_4532Metric -> Fuse:Fuse_1812_4532Metric; P/N MF-MSMF050-2 -> (none); Productor Bourns -> (none); Provider RS -> Mouser; ProviderCode 647-8156 -> 652-MF-MSMF050-2
- P2: renamed from P4; footprint (none) -> Connector_PinHeader_2.54mm:PinHeader_2x03_P2.54mm_Vertical; Manufacturer (none) -> Molex; Provider (none) -> Mouser; ProviderCode (none) -> 538-87914-0616; manf# (none) -> 87914-0616
- P3: renamed from P5; footprint (none) -> Connector_USB:USB_Micro-B_Amphenol_10103594-0001LF_Horizontal; Manufacturer (none) -> Amphenol; Provider (none) -> Mouser; ProviderCode (none) -> 649-10103594-0001LF; manf# (none) -> 10103594-0001LF
- P4: renamed from P6; P/N 53047-0310 -> (none); Productor Molex -> (none); Provider (none) -> Mouser; ProviderCode (none) -> 538-53047-0310
- R1: renamed from R14; Manufacturer (none) -> Vishay; P/N CRCW0603332RFKEA -> (none); Productor Vishay -> (none); Provider (none) -> Mouser; ProviderCode (none) -> 71-CRCW040210K0FKEDC; manf# (none) -> CRCW040210K0FKEDC
- R10: renamed from R24; value R DNM -> 0R DNM; footprint Resistor_SMD:R_0603_1608Metric -> Resistor_SMD:R_0402_1005Metric; Manufacturer (none) -> Vishay; Provider (none) -> Mouser; ProviderCode (none) -> 71-RCC04020000Z0ED; manf# (none) -> RCC04020000Z0ED
- R12: renamed from R25; footprint Resistor_SMD:R_0603_1608Metric -> Resistor_SMD:R_0402_1005Metric; Manufacturer Panasonic -> Yageo; P/N ERJU03F22R0V -> (none); Productor Panasonic -> (none); Provider (none) -> Mouser; ProviderCode (none) -> 603-RC0402FR-0722RL; manf# ERJU03F22R0V -> RC0402FR-0722RL
- R13: renamed from R26; footprint Resistor_SMD:R_0603_1608Metric -> Resistor_SMD:R_0402_1005Metric; Manufacturer Panasonic -> Yageo; P/N ERJU03F22R0V -> (none); Productor Panasonic -> (none); Provider (none) -> Mouser; ProviderCode (none) -> 603-RC0402FR-0722RL; manf# ERJU03F22R0V -> RC0402FR-0722RL
- R14: renamed from R27; value R DNM -> 0R DNM; footprint Resistor_SMD:R_0603_1608Metric -> Resistor_SMD:R_0402_1005Metric; Manufacturer (none) -> Vishay; Provider (none) -> Mouser; ProviderCode (none) -> 71-RCC04020000Z0ED; manf# (none) -> RCC04020000Z0ED
- R15: renamed from R28; value R DNM -> 0R DNM; footprint Resistor_SMD:R_0603_1608Metric -> Resistor_SMD:R_0402_1005Metric; Manufacturer (none) -> Vishay; Provider (none) -> Mouser; ProviderCode (none) -> 71-RCC04020000Z0ED; manf# (none) -> RCC04020000Z0ED
- R16: renamed from R29; value R DNM -> 0R DNM; footprint Resistor_SMD:R_0603_1608Metric -> Resistor_SMD:R_0402_1005Metric; Manufacturer (none) -> Vishay; Provider (none) -> Mouser; ProviderCode (none) -> 71-RCC04020000Z0ED; manf# (none) -> RCC04020000Z0ED
- R17: renamed from R30; value R DNM -> 0R DNM; footprint Resistor_SMD:R_0603_1608Metric -> Resistor_SMD:R_0402_1005Metric; Manufacturer (none) -> Vishay; Provider (none) -> Mouser; ProviderCode (none) -> 71-RCC04020000Z0ED; manf# (none) -> RCC04020000Z0ED
- R2: renamed from R16; footprint Resistor_SMD:R_0603_1608Metric -> Resistor_SMD:R_0402_1005Metric; Manufacturer (none) -> Vishay; P/N CRCW0603332RFKEA -> (none); Productor Vishay -> (none); Provider (none) -> Mouser; ProviderCode (none) -> 71-CRCW04021K00FKEDC; manf# (none) -> CRCW04021K00FKEDC
- R4: renamed from R15; value R DNM -> 0R DNM; footprint Resistor_SMD:R_0603_1608Metric -> Resistor_SMD:R_0402_1005Metric; Manufacturer (none) -> Vishay; Provider (none) -> Mouser; ProviderCode (none) -> 71-RCC04020000Z0ED; manf# (none) -> RCC04020000Z0ED
- R5: renamed from R17; value R DNM -> 0R DNM; footprint Resistor_SMD:R_0603_1608Metric -> Resistor_SMD:R_0402_1005Metric; Manufacturer (none) -> Vishay; Provider (none) -> Mouser; ProviderCode (none) -> 71-RCC04020000Z0ED; manf# (none) -> RCC04020000Z0ED
- R6: renamed from R18; value R DNM -> 0R DNM; footprint Resistor_SMD:R_0603_1608Metric -> Resistor_SMD:R_0402_1005Metric; Manufacturer (none) -> Vishay; Provider (none) -> Mouser; ProviderCode (none) -> 71-RCC04020000Z0ED; manf# (none) -> RCC04020000Z0ED
- R7: renamed from R20; value 10k 1% 1/16W -> 10k; Manufacturer (none) -> Vishay; Provider (none) -> Mouser; ProviderCode (none) -> 71-CRCW040210K0FKEDC; manf# (none) -> CRCW040210K0FKEDC
- R8: renamed from R21; value R DNM -> 0R DNM; footprint Resistor_SMD:R_0603_1608Metric -> Resistor_SMD:R_0402_1005Metric; Manufacturer (none) -> Vishay; Provider (none) -> Mouser; ProviderCode (none) -> 71-RCC04020000Z0ED; manf# (none) -> RCC04020000Z0ED
- R9: renamed from R23; value R DNM -> 0R DNM; footprint Resistor_SMD:R_0603_1608Metric -> Resistor_SMD:R_0402_1005Metric; Manufacturer (none) -> Vishay; Provider (none) -> Mouser; ProviderCode (none) -> 71-RCC04020000Z0ED; manf# (none) -> RCC04020000Z0ED
- SW1: footprint (none) -> Button_Switch_SMD:SW_SPST_B3U-1000P; Manufacturer (none) -> Omron; Provider (none) -> Mouser; ProviderCode (none) -> 653-B3U-1000P; manf# (none) -> B3U-1000P
- U1: renamed from U2; footprint (none) -> Package_DFN_QFN:QFN-44-1EP_7x7mm_P0.5mm_EP5.2x5.2mm; P/N ATmega32U4 -> (none); Productor Atmel -> (none); Provider (none) -> Mouser; ProviderCode (none) -> 556-ATMEGA32U4-MU; manf# (none) -> ATmega32U4-MU
- U2: renamed from U3; value ADM3101EACPZ-250R7 -> ADM3101E; footprint (none) -> Driverino:CP-12-4; Manufacturer Analog Devices -> Analog; Provider (none) -> Mouser; ProviderCode (none) -> 584-AM3101EACPZ250R7; manf# (none) -> ADM3101EACPZ-250R7
- Y1: footprint Crystal:Crystal_SMD_2520-4Pin_2.5x2.0mm -> Crystal:Crystal_SMD_2016-4Pin_2.0x1.6mm; P/N XRCHA16M000F0A01R0 -> (none); Productor Murata -> (none); Provider (none) -> Mouser; ProviderCode (none) -> 81-XRCHA16M000F0A1R0
- renumbered L2 to L1
Connections:
- net +5V: now also JP1.1 (A), P1.2 (PM); no longer C1.2, C2.2, C5.1, C9.1, D1.1 (K), L1.1, P2.2, R1.1, R8.2, U1.14 (VCC), U1.2 (UVCC), U1.24 (AVCC), U1.34 (VCC), U2.5 (VCC)
- net D4: now also R11.2
- net GND: now also U1.45 (EP), C15.1, D3.1 (K), P1.1 (P1)
- net VBUS: now also C15.2, JP1.3 (B)
- net TX_LED: now reaches U1.22 (PD5)
- net TX_LED: now also R3.1
- new net: D3.2 (A), R3.2
- new net PWM_IN: P1.3 (P3), R11.1
- new net VCC: C1.2, C2.2, C5.1, C9.1, D1.1 (K), JP1.2 (C), L1.1, P2.2, R1.1, R8.2, U1.14 (VCC), U1.2 (UVCC), U1.24 (AVCC), U1.34 (VCC), U2.5 (VCC)
Other:
- note added: "-"
- note added: "1-2"
- note added: "2-3"
- note added: "JP?"
- note added: "NO"
- note added: "USB"
- note added: "VM"
- note added: "X"
- moved on the sheet: C1, C2, D1, D2, D4, R1, R10, R14, R15, R16, R17, R2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

Commit message: Update
Parts:
- F1: value 0.5A -> 0.2A; footprint Fuse:Fuse_1812_4532Metric -> Fuse:Fuse_1206_3216Metric; ProviderCode 652-MF-MSMF050-2 -> 652-MF-NSMF020X-2; manf# MF-MSMF050-2 -> MF-NSMF020X-2
- JP1: symbol Jumper:Jumper_3_Bridged12 -> Driverino-rescue:Jumper_3_Bridged12-Jumper
Changed lines of the file:
@@
 AR Path="/614792E0/614921EC" Ref="F1"  Part="1"
 F 0 "F1" H 12925 5492 40  0000 C CNN
-F 1 "0.5A " H 12925 5416 40  0000 C CNN
-F 2 "Fuse:Fuse_1812_4532Metric" H 12925 5275 60  0001 C CNN
+F 1 "0.2A " H 12925 5416 40  0000 C CNN
+F 2 "Fuse:Fuse_1206_3216Metric" H 12925 5275 60  0001 C CNN
 F 3 "" H 12925 5275 60  0001 C CNN
 F 4 "Bourns" H 12925 5275 50  0001 C CNN "Manufacturer"
-F 5 "" H 12925 5275 50  0001 C CNN "P/N"
-F 6 "652-MF-MSMF050-2" H 12925 5275 50  0001 C CNN "ProviderCode"
-F 7 "Mouser" H 12925 5275 50  0001 C CNN "Provider"
-F 8 "MF-MSMF050-2" H 12925 5275 50  0001 C CNN "manf#"
-F 9 "" H 12925 5275 50  0001 C CNN "Productor"
+F 5 "652-MF-NSMF020X-2" H 12925 5275 50  0001 C CNN "ProviderCode"
+F 6 "Mouser" H 12925 5275 50  0001 C CNN "Provider"
+F 7 "MF-NSMF020X-2" H 12925 5275 50  0001 C CNN "manf#"
+F 8 "" H 12925 5275 50  0001 C CNN "Productor"
 	1    12925 5275
 	1    0    0    -1
@@
 $EndComp
 $Comp
-L Jumper:Jumper_3_Bridged12 JP?
+L Driverino-rescue:Jumper_3_Bridged12-Jumper JP?
 U 1 1 609E3044
 P 13900 2075

Commit message: Update
Parts:
- removed R10, R14, R15, R16, R17, R9: 0R DNM, Resistor_SMD:R_0402_1005Metric, symbol Driverino-rescue:R-device
- D4: footprint Diode_SMD:D_SOD-123 -> Diode_SMD:D_0603_1608Metric; ProviderCode 771-BZT52-C4V7X -> 771-BZX884S-C5V1YL; manf# BZT52-C4V7X -> BZX884S-C5V1YL
Connections:
- net D10 is gone; now on net CS2: U1.30 (PB6)
- net D12 is gone; now on net FAULT: U1.26 (PD6)
- net D5 is gone; now on net DRVOFF: U1.31 (PC6)
- net D6 is gone; now on net FGOUT: U1.27 (PD7)
- net D8 is gone; now on net PWM: U1.28 (PB4)
- net D9 is gone; now on net BRAKE: U1.29 (PB5)
Changed lines of the file:
@@
 Text Label 13250 8525 2    50   ~ 0
 D6
-Text HLabel 12650 7950 2    50   Input ~ 0
+Text HLabel 13375 8525 2    50   Input ~ 0
 FGOUT
-$Comp
-L Driverino-rescue:R-device R?
-U 1 1 61658E20
-P 13625 7650
-AR Path="/61658E20" Ref="R?"  Part="1"
-AR Path="/614792E0/61658E20" Ref="R14"  Part="1"
-F 0 "R14" V 13440 7650 40  0000 C CNN
-F 1 "0R DNM" V 13516 7650 40  0000 C CNN
-F 2 "Resistor_SMD:R_0402_1005Metric" V 13555 7650 30  0001 C CNN
-F 3 "" H 13625 7650 30  0000 C CNN
-F 4 "Mouser" H 13625 7650 50  0001 C CNN "Provider"
-F 5 "Vishay" H 13625 7650 50  0001 C CNN "Manufacturer"
-F 6 "71-RCC04020000Z0ED" H 13625 7650 50  0001 C CNN "ProviderCode"
-F 7 "RCC04020000Z0ED" H 13625 7650 50  0001 C CNN "manf#"
-	1    13625 7650
-	0    1    1    0
-$EndComp
-Wire Wire Line
-	13250 7650 13375 7650
-Wire Wire Line
-	13875 7650 14025 7650
-Text HLabel 14025 7650 2    50   Output ~ 0
+Text HLabel 13375 7650 2    50   Output ~ 0
 CS2
-$Comp
-L Driverino-rescue:R-device R?
-U 1 1 61663BE3
-P 13625 7950
-AR Path="/61663BE3" Ref="R?"  Part="1"
-AR Path="/614792E0/61663BE3" Ref="R15"  Part="1"
-F 0 "R15" V 13440 7950 40  0000 C CNN
-F 1 "0R DNM" V 13516 7950 40  0000 C CNN
-F 2 "Resistor_SMD:R_0402_1005Metric" V 13555 7950 30  0001 C CNN
-F 3 "" H 13625 7950 30  0000 C CNN
-F 4 "Mouser" H 13625 7950 50  0001 C CNN "Provider"
-F 5 "Vishay" H 13625 7950 50  0001 C CNN "Manufacturer"
-F 6 "71-RCC04020000Z0ED" H 13625 7950 50  0001 C CNN "ProviderCode"
-F 7 "RCC04020000Z0ED" H 13625 7950 50  0001 C CNN "manf#"
-	1    13625 7950
-	0    1    1    0
-$EndComp
 Wire Wire Line
 	13250 7950 13375 7950
-Wire Wire Line
-	13875 7950 14025 7950
-Text HLabel 14025 7950 2    50   Output ~ 0
+Text HLabel 12150 7950 2    50   Output ~ 0
 DRVOFF
-$Comp
-L Driverino-rescue:R-device R?
-U 1 1 61663BF1
-P 13625 8250
-AR Path="/61663BF1" Ref="R?"  Part="1"
-AR Path="/614792E0/61663BF1" Ref="R16"  Part="1"
-F 0 "R16" V 13440 8250 40  0000 C CNN
-F 1 "0R DNM" V 13516 8250 40  0000 C CNN
-F 2 "Resistor_SMD:R_0402_1005Metric" V 13555 8250 30  0001 C CNN
-F 3 "" H 13625 8250 30  0000 C CNN
-F 4 "Mouser" H 13625 8250 50  0001 C CNN "Provider"
-F 5 "Vishay" H 13625 8250 50  0001 C CNN "Manufacturer"
-F 6 "71-RCC04020000Z0ED" H 13625 8250 50  0001 C CNN "ProviderCode"
-F 7 "RCC04020000Z0ED" H 13625 8250 50  0001 C CNN "manf#"
-	1    13625 8250
-	0    1    1    0
-$EndComp
 Wire Wire Line
 	13250 8250 13375 8250
-Wire Wire Line
-	13875 8250 14025 8250
-Text HLabel 14025 8250 2    50   Output ~ 0
+Text HLabel 13375 8250 2    50   Output ~ 0
 PWM
-$Comp
-L Driverino-rescue:R-device R?
-U 1 1 6166E2E1
-P 13625 8525
-AR Path="/6166E2E1" Ref="R?"  Part="1"
-AR Path="/614792E0/6166E2E1" Ref="R17"  Part="1"
-F 0 "R17" V 13440 8525 40  0000 C CNN
-F 1 "0R DNM" V 13516 8525 40  0000 C CNN
-F 2 "Resistor_SMD:R_0402_1005Metric" V 13555 8525 30  0001 C CNN
-F 3 "" H 13625 8525 30  0000 C CNN
-F 4 "Mouser" H 13625 8525 50  0001 C CNN "Provider"
-F 5 "Vishay" H 13625 8525 50  0001 C CNN "Manufacturer"
-F 6 "71-RCC04020000Z0ED" H 13625 8525 50  0001 C CNN "ProviderCode"
-F 7 "RCC04020000Z0ED" H 13625 8525 50  0001 C CNN "manf#"
-	1    13625 8525
-	0    1    1    0
-$EndComp
 Wire Wire Line
 	13250 8525 13375 8525
-Wire Wire Line
-	13875 8525 14025 8525
-Text HLabel 14025 8525 2    50   Output ~ 0
+Text HLabel 13375 7950 2    50   Output ~ 0
 BRAKE
-Text HLabel 12650 7650 2    50   Input ~ 0
+Text HLabel 12150 7650 2    50   Input ~ 0
 FAULT
 Wire Wire Line
@@
 Text Label 11875 7650 2    50   ~ 0
 D12
-Wire Wire Line
-	12500 7650 12650 7650
-Wire Wire Line
-	11875 7650 12000 7650
-$Comp
-L Driverino-rescue:R-device R?
-U 1 1 616A9031
-P 12250 7650
-AR Path="/616A9031" Ref="R?"  Part="1"
-AR Path="/614792E0/616A9031" Ref="R9"  Part="1"
-F 0 "R9" V 12065 7650 40  0000 C CNN
-F 1 "0R DNM" V 12141 7650 40  0000 C CNN
-F 2 "Resistor_SMD:R_0402_1005Metric" V 12180 7650 30  0001 C CNN
-F 3 "" H 12250 7650 30  0000 C CNN
-F 4 "Mouser" H 12250 7650 50  0001 C CNN "Provider"
-F 5 "Vishay" H 12250 7650 50  0001 C CNN "Manufacturer"
-F 6 "71-RCC04020000Z0ED" H 12250 7650 50  0001 C CNN "ProviderCode"
-F 7 "RCC04020000Z0ED" H 12250 7650 50  0001 C CNN "manf#"
-	1    12250 7650
-	0    1    1    0
-$EndComp
-Wire Wire Line
-	12500 7950 12650 7950
-Wire Wire Line
-	11875 7950 12000 7950
-$Comp
-L Driverino-rescue:R-device R?
-U 1 1 61643BD7
-P 12250 7950
-AR Path="/61643BD7" Ref="R?"  Part="1"
-AR Path="/614792E0/61643BD7" Ref="R10"  Part="1"
-F 0 "R10" V 12065 7950 40  0000 C CNN
-F 1 "0R DNM" V 12141 7950 40  0000 C CNN
-F 2 "Resistor_SMD:R_0402_1005Metric" V 12180 7950 30  0001 C CNN
-F 3 "" H 12250 7950 30  0000 C CNN
-F 4 "Mouser" H 12250 7950 50  0001 C CNN "Provider"
-F 5 "Vishay" H 12250 7950 50  0001 C CNN "Manufacturer"
-F 6 "71-RCC04020000Z0ED" H 12250 7950 50  0001 C CNN "ProviderCode"
-F 7 "RCC04020000Z0ED" H 12250 7950 50  0001 C CNN "manf#"
-	1    12250 7950
-	0    1    1    0
-$EndComp
 Text Label 11875 7950 2    50   ~ 0
 D5
@@
 F 0 "D4" V 8405 9556 40  0000 R CNN
 F 1 "VZ=5V" V 8337 9556 30  0000 R CNN
-F 2 "Diode_SMD:D_SOD-123" V 8325 9550 60  0001 R CNN
+F 2 "Diode_SMD:D_0603_1608Metric" V 8325 9550 60  0001 R CNN
 F 3 "" H 8375 9625 60  0000 C CNN
 F 4 "Mouser" H 8375 9625 50  0001 C CNN "Provider"
 F 5 "" H 8375 9625 50  0001 C CNN "Code"
-F 6 "" H 8375 9625 50  0001 C CNN "P/N"
-F 7 "" H 8375 9625 50  0001 C CNN "Productor"
-F 8 "BZT52-C4V7X" H 8375 9625 50  0001 C CNN "manf#"
-F 9 "Nexperia" H 8375 9625 50  0001 C CNN "Manufacturer"
-F 10 "771-BZT52-C4V7X" H 8375 9625 50  0001 C CNN "ProviderCode"
+F 6 "" H 8375 9625 50  0001 C CNN "Productor"
+F 7 "BZX884S-C5V1YL" H 8375 9625 50  0001 C CNN "manf#"
+F 8 "Nexperia" H 8375 9625 50  0001 C CNN "Manufacturer"
+F 9 "771-BZX884S-C5V1YL" H 8375 9625 50  0001 C CNN "ProviderCode"
 	1    8375 9625
 	0    -1   -1   0
@@
 Text Label 11875 8250 2    50   ~ 0
 D4
+Wire Wire Line
+	11875 7950 12150 7950
+Wire Wire Line
+	13250 7650 13375 7650
+Wire Wire Line
+	11875 7650 12150 7650
 $EndSCHEMATC

Commit message: Modified F1
Parts:
- removed D4: VZ=5V, Diode_SMD:D_0603_1608Metric, symbol Driverino-rescue:ZENERsmall-device
- removed R5, R6: 0R DNM, Resistor_SMD:R_0402_1005Metric, symbol Driverino-rescue:R-device
- F1: value 0.2A -> 200mA; footprint Fuse:Fuse_1206_3216Metric -> Fuse:Fuse_0402_1005Metric; ProviderCode 652-MF-NSMF020X-2 -> 652-MF-ASML020/6-2; manf# MF-NSMF020X-2 -> MF-ASML020/6-2
Connections:
- net A0: now also C6.2, R4.1
- net A5: no longer C6.2, R4.1
Changed lines of the file:
@@
 Wire Wire Line
 	14225 4650 14050 4650
-Text Label 6500 9275 2    50   ~ 0
-A5
 Wire Wire Line
 	5150 9275 5350 9275
@@
 AR Path="/614792E0/614921EC" Ref="F1"  Part="1"
 F 0 "F1" H 12925 5492 40  0000 C CNN
-F 1 "0.2A " H 12925 5416 40  0000 C CNN
-F 2 "Fuse:Fuse_1206_3216Metric" H 12925 5275 60  0001 C CNN
+F 1 "200mA" H 12925 5416 40  0000 C CNN
+F 2 "Fuse:Fuse_0402_1005Metric" H 12925 5275 60  0001 C CNN
 F 3 "" H 12925 5275 60  0001 C CNN
 F 4 "Bourns" H 12925 5275 50  0001 C CNN "Manufacturer"
-F 5 "652-MF-NSMF020X-2" H 12925 5275 50  0001 C CNN "ProviderCode"
+F 5 "652-MF-ASML020/6-2" H 12925 5275 50  0001 C CNN "ProviderCode"
 F 6 "Mouser" H 12925 5275 50  0001 C CNN "Provider"
-F 7 "MF-NSMF020X-2" H 12925 5275 50  0001 C CNN "manf#"
+F 7 "MF-ASML020/6-2" H 12925 5275 50  0001 C CNN "manf#"
 F 8 "" H 12925 5275 50  0001 C CNN "Productor"
 	1    12925 5275
@@
 Wire Wire Line
 	12550 5375 12550 5275
-Wire Wire Line
-	7150 9075 7150 9275
-$Comp
-L power:HT #PWR?
-U 1 1 614922C9
-P 7150 9075
-AR Path="/614922C9" Ref="#PWR?"  Part="1"
-AR Path="/614792E0/614922C9" Ref="#PWR013"  Part="1"
-F 0 "#PWR013" H 7150 9195 20  0001 C CNN
-F 1 "HT" H 7170 9211 40  0000 C CNN
-F 2 "" H 7150 9075 50  0001 C CNN
-F 3 "" H 7150 9075 50  0001 C CNN
-	1    7150 9075
-	1    0    0    -1
-$EndComp
 Text Label 14050 4650 0    50   ~ 0
 RESET
@@
 Wire Wire Line
 	12250 5875 12250 5950
-Text Label 10875 9275 2    50   ~ 0
-A3
 Wire Wire Line
 	9500 9275 9800 9275
@@
 	12250 5875 12550 5875
 Wire Wire Line
-	8375 9900 8375 10050
-Connection ~ 8375 9900
-Wire Wire Line
-	8000 9900 8375 9900
-Wire Wire Line
-	8000 9850 8000 9900
-Wire Wire Line
-	8000 9275 8375 9275
-Connection ~ 8000 9275
-Wire Wire Line
-	8000 9350 8000 9275
-Connection ~ 8375 9275
-Wire Wire Line
-	8375 9275 8725 9275
-$Comp
-L Driverino-rescue:R-device R?
-U 1 1 614920AF
-P 8000 9600
-AR Path="/614920AF" Ref="R?"  Part="1"
-AR Path="/614792E0/614920AF" Ref="R6"  Part="1"
-F 0 "R6" H 7929 9562 40  0000 R CNN
-F 1 "0R DNM" H 7929 9638 40  0000 R CNN
-F 2 "Resistor_SMD:R_0402_1005Metric" V 7930 9600 30  0001 C CNN
-F 3 "" H 8000 9600 30  0000 C CNN
-F 4 "Mouser" H 8000 9600 50  0001 C CNN "Provider"
-F 5 "Vishay" H 8000 9600 50  0001 C CNN "Manufacturer"
-F 6 "71-RCC04020000Z0ED" H 8000 9600 50  0001 C CNN "ProviderCode"
-F 7 "RCC04020000Z0ED" H 8000 9600 50  0001 C CNN "manf#"
-	1    8000 9600
-	-1   0    0    1
-$EndComp
-Wire Wire Line
-	8375 9725 8375 9900
-Wire Wire Line
-	8375 9275 8375 9525
-$Comp
-L Driverino-rescue:ZENERsmall-device D?
-U 1 1 6149209F
-P 8375 9625
-AR Path="/6149209F" Ref="D?"  Part="1"
-AR Path="/614792E0/6149209F" Ref="D4"  Part="1"
-F 0 "D4" V 8405 9556 40  0000 R CNN
-F 1 "VZ=5V" V 8337 9556 30  0000 R CNN
-F 2 "Diode_SMD:D_0603_1608Metric" V 8325 9550 60  0001 R CNN
-F 3 "" H 8375 9625 60  0000 C CNN
-F 4 "Mouser" H 8375 9625 50  0001 C CNN "Provider"
-F 5 "" H 8375 9625 50  0001 C CNN "Code"
-F 6 "" H 8375 9625 50  0001 C CNN "Productor"
-F 7 "BZX884S-C5V1YL" H 8375 9625 50  0001 C CNN "manf#"
-F 8 "Nexperia" H 8375 9625 50  0001 C CNN "Manufacturer"
-F 9 "771-BZX884S-C5V1YL" H 8375 9625 50  0001 C CNN "ProviderCode"
-	1    8375 9625
-	0    -1   -1   0
-$EndComp
-$Comp
-L Driverino-rescue:GND-power #PWR?
-U 1 1 61492093
-P 8375 10050
-AR Path="/61492093" Ref="#PWR?"  Part="1"
-AR Path="/614792E0/61492093" Ref="#PWR017"  Part="1"
-F 0 "#PWR017" H 8375 10050 30  0001 C CNN
-F 1 "GND" H 8375 9980 30  0001 C CNN
-F 2 "" H 8375 10050 50  0001 C CNN
-F 3 "" H 8375 10050 50  0001 C CNN
-	1    8375 10050
-	1    0    0    -1
-$EndComp
-Text Label 8725 9275 2    50   ~ 0
-A4
-Wire Wire Line
-	7150 9275 7325 9275
-Wire Wire Line
-	7825 9275 8000 9275
-$Comp
-L Driverino-rescue:R-device R?
-U 1 1 614920A8
-P 7575 9275
-AR Path="/614920A8" Ref="R?"  Part="1"
-AR Path="/614792E0/614920A8" Ref="R5"  Part="1"
-F 0 "R5" V 7390 9275 40  0000 C CNN
-F 1 "0R DNM" V 7466 9275 40  0000 C CNN
-F 2 "Resistor_SMD:R_0402_1005Metric" V 7505 9275 30  0001 C CNN
-F 3 "" H 7575 9275 30  0000 C CNN
-F 4 "Mouser" H 7575 9275 50  0001 C CNN "Provider"
-F 5 "Vishay" H 7575 9275 50  0001 C CNN "Manufacturer"
-F 6 "71-RCC04020000Z0ED" H 7575 9275 50  0001 C CNN "ProviderCode"
-F 7 "RCC04020000Z0ED" H 7575 9275 50  0001 C CNN "manf#"
-	1    7575 9275
-	0    1    1    0
-$EndComp
-Wire Wire Line
 	7350 6375 7350 6575
 Wire Wire Line
@@
 Wire Wire Line
 	11875 7650 12150 7650
+Text Label 10875 9275 2    50   ~ 0
+A3
+Text Label 6500 9275 2    50   ~ 0
+A0
 $EndSCHEMATC
