File: ARDUINO-MICRO.sch (KiCad schematic (older format))
At the start: 39 parts, among them P1 RC_IN, P2 ICSP, P3 USB-MICRO, P4 RS232, SW1 SW_PUSH, U1 ATmega32U4, U2 ADM3101E, Y1 16MHz

Commit message: Update
Parts:
- JP1: footprint Driverino:TDD01H0SB1R -> Connector_PinHeader_1.27mm:PinHeader_1x03_P1.27mm_Vertical; Manufacturer C&K -> Samtec; ProviderCode 611-TDD01H0SB1R -> 200-TMS10301GS; manf# TDD01H0SB1R -> TMS-103-01-G-S
Changed lines of the file:
@@
 F 0 "JP1" H 13900 2179 40  0000 C CNN
 F 1 "VCC_SEL" H 13900 2255 40  0000 C CNN
-F 2 "Driverino:TDD01H0SB1R" H 13900 2075 50  0001 C CNN
+F 2 "Connector_PinHeader_1.27mm:PinHeader_1x03_P1.27mm_Vertical" H 13900 2075 50  0001 C CNN
 F 3 "~" H 13900 2075 50  0001 C CNN
-F 4 "	C&K" H 13900 2075 50  0001 C CNN "Manufacturer"
+F 4 "Samtec" H 13900 2075 50  0001 C CNN "Manufacturer"
 F 5 "Mouser" H 13900 2075 50  0001 C CNN "Provider"
-F 6 "611-TDD01H0SB1R" H 13900 2075 50  0001 C CNN "ProviderCode"
-F 7 "TDD01H0SB1R" H 13900 2075 50  0001 C CNN "manf#"
+F 6 "200-TMS10301GS" H 13900 2075 50  0001 C CNN "ProviderCode"
+F 7 "TMS-103-01-G-S" H 13900 2075 50  0001 C CNN "manf#"
 	1    13900 2075
 	-1   0    0    1
