File: Driverino.kicad_pcb (KiCad board)
At the start: 2 copper layers, 25 x 40 mm, 82 parts, among them P1 RC_IN, P2 ICSP, P3 USB-MICRO, P4 RS232, P5 PWR_IN, P6 HALL, P7 MOT, SW1 SW_PUSH, U1 ATmega32U4, U2 ADM3101E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

Commit message: Update
Parts:
- C1, C12, C13, C15, C16, C18, C2, C20, C3, C4, C5, C7, C9, D1, L1, R1, R22, R23, R5, R6: moved to B.Cu
- F1: footprint Fuse:Fuse_1812_4532Metric -> Fuse:Fuse_1206_3216Metric
- moved C18 113.4 mm to (163.5, 86.9)
- moved C22 95.6 mm to (148.2, 93.0), turned to 90 degrees
- moved C20 92.9 mm to (162.8, 83.6)
- moved R22 86.8 mm to (143.6, 92.0), turned to 180 degrees
- moved R23 84.7 mm to (137.4, 92.0)
- moved R5 80.0 mm to (171.5, 89.7), turned to 90 degrees
- moved R6 74.7 mm to (175.5, 89.9), turned to 90 degrees
- moved C2 65.8 mm to (153.5, 101.0)
- moved L2 64.9 mm to (145.5, 90.3), turned to 270 degrees
- moved D1 64.3 mm to (153.5, 99.0), turned to 180 degrees
- moved C1 62.6 mm to (153.5, 102.0)
- moved L1 59.2 mm to (138.2, 103.0), turned to 90 degrees
- moved C12 57.0 mm to (149.2, 96.5), turned to 180 degrees
- moved C4 56.6 mm to (139.9, 103.2), turned to 90 degrees
- moved C10 55.6 mm to (147.3, 100.7)
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Connections:
- P5 pad 1: GNDPWR -> HT
- P5 pad 2: HT -> GNDPWR
Routing:
- net /ARDUINO-MICRO/MOSI: track 0.00 -> 30.4 mm, vias 0 -> 2
- net /ARDUINO-MICRO/MISO: track 0.00 -> 30.3 mm, vias 0 -> 2
- net /ARDUINO-MICRO/SCK: track 0.00 -> 23.8 mm, vias 0 -> 2
- net VBUS: track 0.00 -> 12.6 mm, vias 0 -> 2
- net /ARDUINO-MICRO/D-: track 0.00 -> 10.2 mm
- net /ARDUINO-MICRO/D+: track 0.00 -> 9.45 mm
- net /ARDUINO-MICRO/RESET: track 0.00 -> 7.45 mm
- net VCC: track 0.00 -> 6.18 mm, vias 0 -> 1
- net Net-(C10-Pad1): track 0.00 -> 3.48 mm
- net Net-(C11-Pad1): track 0.00 -> 3.48 mm
- net Net-(C4-Pad2): track 0.00 -> 3.17 mm, vias 0 -> 1
- net Net-(C3-Pad2): track 0.00 -> 2.97 mm, vias 0 -> 1
- net Net-(R7-Pad2): track 0.00 -> 2.24 mm
- net Net-(P3-Pad3): track 0.00 -> 2.15 mm
- net Net-(P3-Pad2): track 0.00 -> 2.15 mm
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- added copper zone on F.Cu, net /DRIVER/FB
- added copper zone on F.Cu, net /DRIVER/SW
- added copper zone on F.Cu, net /DRIVER/U
- added copper zone on F.Cu, net /DRIVER/V
- added copper zone on F.Cu, net /DRIVER/W
- added copper zone on B.Cu, net GND
- added copper zone on F.Cu, net GND
- added copper zone on B.Cu, net GNDPWR
- added copper zone on F.Cu, net GNDPWR
- added copper zone on F.Cu, net HT
Other:
- board size 25 x 40 mm -> 25 x 41 mm
- board text added: "TODO: U3 pads size, Y1 pins"

Commit message: Update
Parts:
- removed R10, R14, R15, R16, R17, R9: 0R DNM, Resistor_SMD:R_0402_1005Metric
- C14, C23, C24, C25, C26, C6, R11, R18, R19, R2, R20, R21, R24, R25, R27, R28, R29, R3, R30: moved to B.Cu
- C18, C20: moved to F.Cu
- D4: footprint Diode_SMD:D_SOD-123 -> Diode_SMD:D_0603_1608Metric; moved to B.Cu
- JP1: footprint Driverino:TDD01H0SB1R -> Connector_PinHeader_1.27mm:PinHeader_1x03_P1.27mm_Vertical
- JP2: footprint Driverino:TDD01H0SB1R -> rob-int:3JUMPER_0603; moved to B.Cu
- moved R26 105.6 mm to (157.0, 87.3), turned to 270 degrees
- moved D7 101.9 mm to (156.5, 77.6), turned to 270 degrees
- moved D5 92.7 mm to (134.2, 78.4), turned to 180 degrees
- moved D8 92.4 mm to (134.3, 81.4)
- moved D4 91.2 mm to (154.2, 89.0), turned to 270 degrees
- moved R21 88.4 mm to (134.4, 81.4), turned to 180 degrees
- moved R20 87.9 mm to (156.5, 79.2), turned to 90 degrees
- moved R27 83.6 mm to (137.0, 91.1), turned to 90 degrees
- moved R18 82.7 mm to (134.4, 78.4), turned to 180 degrees
- moved F2 82.4 mm to (147.8, 93.2), turned to 90 degrees
- moved R25 81.2 mm to (133.2, 95.3), turned to 90 degrees
- moved C26 80.2 mm to (135.9, 90.2), turned to 270 degrees
- moved R24 79.5 mm to (137.0, 94.1), turned to 270 degrees
- moved R3 77.8 mm to (156.1, 92.0)
- moved C23 76.0 mm to (134.2, 83.2)
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Connections:
- U1 pad 26: /ARDUINO-MICRO/D12 -> /ARDUINO-MICRO/FAULT
- U1 pad 27: /ARDUINO-MICRO/D6 -> /ARDUINO-MICRO/FGOUT
- U1 pad 28: /ARDUINO-MICRO/D8 -> /ARDUINO-MICRO/PWM
- U1 pad 29: /ARDUINO-MICRO/D9 -> /ARDUINO-MICRO/BRAKE
- U1 pad 30: /ARDUINO-MICRO/D10 -> /ARDUINO-MICRO/CS2
Routing:
- net +3.3V: track 0.00 -> 27.0 mm, vias 0 -> 1
- net /ARDUINO-MICRO/TX_LED: track 0.00 -> 13.0 mm, vias 0 -> 1
- net /ARDUINO-MICRO/RESET: track 7.45 -> 18.9 mm, vias 0 -> 4
- net /DRIVER/HBP: track 0.00 -> 9.25 mm
- net /DRIVER/HBN: track 0.00 -> 8.93 mm
- net /DRIVER/HCN: track 0.00 -> 8.35 mm
- net /DRIVER/HAP: track 0.00 -> 7.59 mm
- net /DRIVER/HCP: track 0.00 -> 7.53 mm
- net HT: track 0.00 -> 7.48 mm, vias 2 -> 1
- net /DRIVER/HAN: track 0.00 -> 6.84 mm
- net /ARDUINO-MICRO/TXO: track 0.00 -> 5.52 mm
- net /ARDUINO-MICRO/FGOUT: track 0.00 -> 5.32 mm, vias 0 -> 1
- net /ARDUINO-MICRO/RXI: track 0.00 -> 4.82 mm, vias 0 -> 2
- net /ARDUINO-MICRO/CS2: track 0.00 -> 3.86 mm
- net /ARDUINO-MICRO/PWM: track 0.00 -> 3.47 mm
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- removed copper zone on B.Cu, net GNDPWR
Other:
- board size 25 x 41 mm -> 26 x 41 mm
- net class Default: clearance 0.2 -> 0.15
- rule trace_clearance: 0.2 -> 0.15
- rule trace_min: 0.2 -> 0.15
- rule via_min_drill: 0.3 -> 0.2
- rule via_min_size: 0.4 -> 0.5

Commit message: update
Parts:
- moved D3 1.25 mm to (155.8, 93.2)
- moved R3 1.25 mm to (156.1, 93.2)
- moved C23 0.06 mm to (134.2, 83.2)
Routing:
- net /ARDUINO-MICRO/ILIM: track 0.00 -> 11.7 mm, vias 0 -> 2
- net +3.3V: track 27.0 -> 25.7 mm
- net /ARDUINO-MICRO/TX_LED: track 13.0 -> 11.8 mm

Commit message: Routing completed
Parts:
- removed D4: VZ=5V, Diode_SMD:D_0603_1608Metric
- removed R5, R6: 0R DNM, Resistor_SMD:R_0402_1005Metric
- JP2: moved to F.Cu
- moved C6 2.20 mm to (137.3, 97.2)
- moved R4 2.20 mm to (137.3, 97.2)
- moved R20 2.10 mm to (156.2, 77.2), turned to 0 degrees
- moved JP1 0.80 mm to (133.8, 102.8)
- moved D7 0.72 mm to (155.9, 77.2), turned to 0 degrees
- moved P3 0.70 mm to (136.3, 114.2)
- moved JP2 0.67 mm to (134.4, 85.5)
- moved C9 0.62 mm to (150.7, 98.7), turned to 90 degrees
- moved C2 0.56 mm to (148.5, 108.0)
- moved C1 0.50 mm to (147.6, 108.0)
- moved D1 0.50 mm to (145.5, 108.0)
- moved R1 0.50 mm to (146.6, 108.0)
- moved SW1 0.50 mm to (146.6, 108.0)
- moved R19 0.23 mm to (156.0, 103.3), turned to 0 degrees
- moved R2 0.19 mm to (156.0, 101.7), turned to 0 degrees
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Connections:
- C6 pad 2: /ARDUINO-MICRO/A5 -> /ARDUINO-MICRO/A0
- R4 pad 1: /ARDUINO-MICRO/A5 -> /ARDUINO-MICRO/A0
Routing:
- net VCC: track 9.56 -> 89.4 mm, vias 2 -> 7
- net +5V: track 0.00 -> 61.0 mm, vias 0 -> 4
- net /ARDUINO-MICRO/FAULT: track 0.00 -> 31.9 mm, vias 0 -> 3
- net /ARDUINO-MICRO/D4: track 0.00 -> 17.8 mm, vias 0 -> 3
- net /ARDUINO-MICRO/CS1: track 0.00 -> 16.8 mm, vias 0 -> 1
- net Net-(F1-Pad2): track 0.00 -> 3.84 mm
- net /ARDUINO-MICRO/A4: track 2.55 -> 0.00 mm
- net /ARDUINO-MICRO/ILIM: track 11.7 -> 10.0 mm
- net /ARDUINO-MICRO/A5: track 1.58 -> 0.00 mm, vias 1 -> 0
- net /ARDUINO-MICRO/A0: track 0.00 -> 1.46 mm, vias 0 -> 1
- net HT: track 7.48 -> 8.30 mm, vias 1 -> 0
- net /ARDUINO-MICRO/D-: track 10.2 -> 9.38 mm
- net Net-(P3-Pad3): track 2.15 -> 2.85 mm
- net Net-(P3-Pad2): track 2.15 -> 2.85 mm
- net Net-(JP2-Pad2): track 2.25 -> 2.91 mm
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Other:
- board text added: "F1, F2 size, ANALOG INPUTS"
- board text removed: "TODO: U3 pads size, Y1 pins"

Commit message: Gerber plot
Connections:
- U1 pad 31: /ARDUINO-MICRO/D5 -> /ARDUINO-MICRO/DRVOFF
Routing:
- net /ARDUINO-MICRO/FAULT: track 31.9 -> 32.8 mm
- net VCC: track 89.4 -> 89.9 mm
Other:
- board text added: "F1, F2 size, ANALOG INPUTS, DRIVEROFF"
- board text removed: "F1, F2 size, ANALOG INPUTS"

Commit message: Modified F1
Parts:
- F1: footprint Fuse:Fuse_1206_3216Metric -> Fuse:Fuse_0402_1005Metric
- moved F1 1.42 mm to (133.8, 109.1)
Routing:
- net VBUS: track 15.4 -> 17.8 mm
- net Net-(F1-Pad2): track 3.84 -> 3.33 mm
Changed lines of the file:
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@@
     (thickness 1.6)
     (drawings 7)
-    (tracks 440)
+    (tracks 442)
     (zones 0)
     (modules 73)
@@
     (0 F.Cu signal)
     (31 B.Cu signal)
-    (32 B.Adhes user hide)
+    (32 B.Adhes user)
     (33 F.Adhes user)
-    (34 B.Paste user hide)
-    (35 F.Paste user hide)
-    (36 B.SilkS user hide)
-    (37 F.SilkS user hide)
-    (38 B.Mask user hide)
-    (39 F.Mask user hide)
-    (40 Dwgs.User user hide)
-    (41 Cmts.User user hide)
-    (42 Eco1.User user hide)
-    (43 Eco2.User user hide)
-    (44 Edge.Cuts user hide)
-    (45 Margin user hide)
-    (46 B.CrtYd user hide)
-    (47 F.CrtYd user hide)
-    (48 B.Fab user hide)
-    (49 F.Fab user hide)
+    (34 B.Paste user)
+    (35 F.Paste user)
+    (36 B.SilkS user)
+    (37 F.SilkS user)
+    (38 B.Mask user)
+    (39 F.Mask user)
+    (40 Dwgs.User user)
+    (41 Cmts.User user)
+    (42 Eco1.User user)
+    (43 Eco2.User user)
+    (44 Edge.Cuts user)
+    (45 Margin user)
+    (46 B.CrtYd user)
+    (47 F.CrtYd user)
+    (48 B.Fab user)
+    (49 F.Fab user)
   )
   (setup
-    (last_trace_width 0.15)
+    (last_trace_width 0.25)
     (user_trace_width 0.15)
     (user_trace_width 0.5)
@@
     (pad_to_mask_clearance 0)
     (aux_axis_origin 0 0)
-    (visible_elements 7EF9B67F)
+    (visible_elements 7EFFB67F)
     (pcbplotparams
       (layerselection 0x010fc_ffffffff)
@@
     (add_net VCC)
   )
+  (module Fuse:Fuse_0402_1005Metric (layer F.Cu)
+    (at 133.75 109.1 270)
+    (descr "Fuse SMD 0402 (1005 Metric), square (rectangular) end terminal, IPC_7351 nominal, (Body size source: http://www.tortai-tech.com/upload/download/2011102023233369053.pdf), generated with kicad-footprint-generator")
+    (tags resistor)
+    (attr smd)
+    (fp_text reference F1 (at -1.6 0 180) (layer F.SilkS)
+      (effects (font (size 1 1) (thickness 0.15)))
+    )
+    (fp_text value "0.5A " (at -3 -0.5) (layer F.Fab)
+      (effects (font (size 1 1) (thickness 0.15)))
+    )
+    (fp_text user %R (at 0 0 90) (layer F.Fab)
+      (effects (font (size 1 1) (thickness 0.15)))
+    )
+    (fp_line (start -0.5 0.25) (end -0.5 -0.25) (layer F.Fab) (width 0.1))
+    (fp_line (start -0.5 -0.25) (end 0.5 -0.25) (layer F.Fab) (width 0.1))
+    (fp_line (start 0.5 -0.25) (end 0.5 0.25) (layer F.Fab) (width 0.1))
+    (fp_line (start 0.5 0.25) (end -0.5 0.25) (layer F.Fab) (width 0.1))
+    (fp_line (start -0.93 0.47) (end -0.93 -0.47) (layer F.CrtYd) (width 0.05))
+    (fp_line (start -0.93 -0.47) (end 0.93 -0.47) (layer F.CrtYd) (width 0.05))
+    (fp_line (start 0.93 -0.47) (end 0.93 0.47) (layer F.CrtYd) (width 0.05))
+    (fp_line (start 0.93 0.47) (end -0.93 0.47) (layer F.CrtYd) (width 0.05))
+    (pad 2 smd roundrect (at 0.485 0 270) (size 0.59 0.64) (layers F.Cu F.Paste F.Mask) (roundrect_rratio 0.25)
+      (net 39 "Net-(F1-Pad2)"))
+    (pad 1 smd roundrect (at -0.485 0 270) (size 0.59 0.64) (layers F.Cu F.Paste F.Mask) (roundrect_rratio 0.25)
+      (net 16 VBUS))
+    (model ${KISYS3DMOD}/Fuse.3dshapes/Fuse_0402_1005Metric.wrl
+      (at (xyz 0 0 0))
+      (scale (xyz 1 1 1))
+      (rotate (xyz 0 0 0))
+    )
+  )
   (module rob-int:3JUMPER_0603 (layer F.Cu)
     (at 134.45 85.45 180)
@@
     )
   )
-  (module Fuse:Fuse_1206_3216Metric (layer F.Cu)
-    (at 133.75 107.675 270)
-    (descr "Fuse SMD 1206 (3216 Metric), square (rectangular) end terminal, IPC_7351 nominal, (Body size source: http://www.tortai-tech.com/upload/download/2011102023233369053.pdf), generated with kicad-footprint-generator")
-    (tags resistor)
-    (attr smd)
-    (fp_text reference F1 (at 2.875 0.05 180) (layer F.SilkS)
-      (effects (font (size 1 1) (thickness 0.15)))
-    )
-    (fp_text value "0.5A " (at -3 -0.5) (layer F.Fab)
-      (effects (font (size 1 1) (thickness 0.15)))
-    )
-    (fp_line (start 2.28 1.12) (end -2.28 1.12) (layer F.CrtYd) (width 0.05))
-    (fp_line (start 2.28 -1.12) (end 2.28 1.12) (layer F.CrtYd) (width 0.05))
-    (fp_line (start -2.28 -1.12) (end 2.28 -1.12) (layer F.CrtYd) (width 0.05))
-    (fp_line (start -2.28 1.12) (end -2.28 -1.12) (layer F.CrtYd) (width 0.05))
-    (fp_line (start -0.602064 0.91) (end 0.602064 0.91) (layer F.SilkS) (width 0.12))
-    (fp_line (start -0.602064 -0.91) (end 0.602064 -0.91) (layer F.SilkS) (width 0.12))
-    (fp_line (start 1.6 0.8) (end -1.6 0.8) (layer F.Fab) (width 0.1))
-    (fp_line (start 1.6 -0.8) (end 1.6 0.8) (layer F.Fab) (width 0.1))
-    (fp_line (start -1.6 -0.8) (end 1.6 -0.8) (layer F.Fab) (width 0.1))
-    (fp_line (start -1.6 0.8) (end -1.6 -0.8) (layer F.Fab) (width 0.1))
-    (fp_text user %R (at 0 0 90) (layer F.Fab)
-      (effects (font (size 1 1) (thickness 0.15)))
-    )
-    (pad 2 smd roundrect (at 1.4 0 270) (size 1.25 1.75) (layers F.Cu F.Paste F.Mask) (roundrect_rratio 0.2)
-      (net 39 "Net-(F1-Pad2)"))
-    (pad 1 smd roundrect (at -1.4 0 270) (size 1.25 1.75) (layers F.Cu F.Paste F.Mask) (roundrect_rratio 0.2)
-      (net 16 VBUS))
-    (model ${KISYS3DMOD}/Fuse.3dshapes/Fuse_1206_3216Metric.wrl
-      (at (xyz 0 0 0))
-      (scale (xyz 1 1 1))
-      (rotate (xyz 0 0 0))
-    )
-  )
   (module Driverino:39773-0003 (layer F.Cu)
     (at 140.5 79.3 180)
@@
   (segment (start 133.75 106.275) (end 136.25 106.275) (width 0.25) (layer B.Cu) (net 16) (status 20))
   (segment (start 133.75 106.275) (end 133.75 104.12) (width 0.25) (layer F.Cu) (net 16) (status 30))
+  (segment (start 133.75 107.19) (end 133.75 106.275) (width 0.25) (layer F.Cu) (net 16))
+  (segment (start 133.75 108.615) (end 133.75 107.19) (width 0.25) (layer F.Cu) (net 16))
   (segment (start 155.69 77.175) (end 149.8 77.175) (width 0.15) (layer B.Cu) (net 17) (status 10))
   (segment (start 149 77.975) (end 149 79.25) (width 0.15) (layer B.Cu) (net 17) (status 20))
@@
   (segment (start 136.625 85.775) (end 136.625 86.375) (width 0.15) (layer B.Cu) (net 37))
   (segment (start 135.025 112.385) (end 135.025 111.3) (width 0.25) (layer F.Cu) (net 39) (status 10))
-  (segment (start 133.75 110.025) (end 133.75 109.075) (width 0.25) (layer F.Cu) (net 39) (status 20))
   (segment (start 135.025 111.3) (end 133.75 110.025) (width 0.25) (layer F.Cu) (net 39))
+  (segment (start 133.75 110.025) (end 133.75 109.585) (width 0.25) (layer F.Cu) (net 39))
   (segment (start 153.66 106.25) (end 154.775 105.135) (width 0.25) (layer B.Cu) (net 40) (status 10))
   (segment (start 154.775 105.135) (end 154.775 103.7) (width 0.25) (layer B.Cu) (net 40))
