File: Driverino.kicad_pcb (KiCad board)
At the start: 2 copper layers, 26 x 41 mm, 73 parts, among them P1 RC_IN, P2 ICSP, P3 USB-MICRO, P4 RS232, P5 PWR_IN, P6 HALL, P7 MOT, SW1 SW_PUSH, U1 ATmega32U4, U2 ADM3101E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

Commit message: Update
Parts:
- moved C15 1.95 mm to (136.3, 105.8)
Routing:
- net VBUS: track 17.8 -> 19.4 mm, vias 2 -> 1

Commit message: Update
Parts:
- JP2: footprint rob-int:3JUMPER_0603 -> Connector_PinHeader_1.27mm:PinHeader_1x03_P1.27mm_Vertical
- moved JP2 0.74 mm to (134.4, 84.7), turned to 270 degrees
Routing:
- net /ARDUINO-MICRO/FAULT: track 32.8 -> 31.8 mm
- net Net-(JP2-Pad2): track 2.91 -> 3.71 mm
- net +5V: track 61.5 -> 62.2 mm, vias 4 -> 3
- net +3.3V: vias 2 -> 1

Commit message: Update to KiCAD 8.0
Update to KiCAD 8.0
Other:
- net class Default removed
